File: Control-HW/Drivers.kicad_sch (KiCad schematic)
At the start: 12 parts

Commit message: First revision
Parts:
- removed C? (x2): 100n, C_Capacitor:C_0603, symbol C_Capacitor:C_0603
- removed C? (x2): 470n,100v, C_Capacitor:C_0805, symbol C_Capacitor:C_0805
- removed D? (x3): DSS110U, D_Diode:D_SOD_123, symbol D_Diode:DSS110U
- removed U? (x3): IR2101S, U_IC:SOIC_8, symbol U_Driver:IR2101S
- added C11, C12: 470n,100v, C_Capacitor:C_0805, symbol C_Capacitor:C_0805
- added C8, C9: 100n, C_Capacitor:C_0603, symbol C_Capacitor:C_0603
- added U2, U3, U4: 2EDL8024GXUMA1, U_IC:DFN8_08_4x4_EP, symbol U_Driver:2EDL8024GXUMA1
- gave numbers to parts that had none: 2
Connections:
- net +12V: now also C8.1, C9.1, U2.1 (VCC), U3.1 (VCC), U4.1 (VCC)
- net GATE_AH: now also U2.3 (HOUT)
- net GATE_AL: now also U2.8 (LOUT)
- net GATE_BH: now also U3.3 (HOUT)
- net GATE_BL: now also U3.8 (LOUT)
- net GATE_CH: now also U4.3 (HOUT)
- net GATE_CL: now also U4.8 (LOUT)
- net GND: now also C8.2, C9.2, U2.7 (GND), U2.9 (EP), U3.7 (GND), U3.9 (EP), U4.7 (GND), U4.9 (EP)
- net PHASE_A: now also U2.4 (HSRC)
- net PHASE_B: now also C11.2, U3.4 (HSRC)
- net PHASE_C: now also C12.2, U4.4 (HSRC)
- net PWM_AH: now also U2.5 (HIN)
- net PWM_AL: now also U2.6 (LIN)
- net PWM_BH: now also U3.5 (HIN)
- net PWM_BL: now also U3.6 (LIN)
- net PWM_CH: now also U4.5 (HIN)
- net PWM_CL: now also U4.6 (LIN)
- net at C10.1: now also U2.2 (HBOOT)
- new net: C11.1, U3.2 (HBOOT)
- new net: C12.1, U4.2 (HBOOT)
Other:
- note removed: "Qc = 600nC Target rise time = 500nS Ic (nom) = 1.2A Ic (avg) = 24mA"
- moved on the sheet: C10, C7
