File: Control-HW/Sense.kicad_sch (KiCad schematic)
At the start: 12 parts

Commit message: First revision
Parts:
- gave numbers to parts that had none: 12
Changed lines of the file:
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@@
   (symbol (lib_id "R_Resistor:R_0603") (at 179.07 59.69 90) (unit 1)
     (in_bom yes) (on_board yes)
-    (property "Reference" "R?" (id 0) (at 175.26 55.88 90))
+    (property "Reference" "R12" (id 0) (at 175.26 55.88 90))
     (property "Value" "47K" (id 1) (at 179.07 55.88 90))
     (property "Footprint" "R_Resistor:R_0603" (id 2) (at 179.07 62.23 90)
@@
   (symbol (lib_id "R_Resistor:R_0603") (at 179.07 69.85 90) (unit 1)
     (in_bom yes) (on_board yes)
-    (property "Reference" "R?" (id 0) (at 175.26 67.31 90))
+    (property "Reference" "R13" (id 0) (at 175.26 67.31 90))
     (property "Value" "47K" (id 1) (at 179.07 67.31 90))
     (property "Footprint" "R_Resistor:R_0603" (id 2) (at 179.07 72.39 90)
@@
   (symbol (lib_id "C_Capacitor:C_0603") (at 118.11 64.77 0) (unit 1)
     (in_bom yes) (on_board yes) (fields_autoplaced)
-    (property "Reference" "C?" (id 0) (at 120.4341 63.027 0)
+    (property "Reference" "C14" (id 0) (at 120.4341 63.027 0)
       (effects (font (size 1.27 1.27)) (justify left))
     )
@@
   (symbol (lib_id "R_Resistor:R_0603") (at 88.9 80.01 0) (unit 1)
     (in_bom yes) (on_board yes) (fields_autoplaced)
-    (property "Reference" "R?" (id 0) (at 90.551 78.2607 0)
+    (property "Reference" "R5" (id 0) (at 90.551 78.2607 0)
       (effects (font (size 1.27 1.27)) (justify left))
     )
@@
   (symbol (lib_id "R_Resistor:R_0603") (at 179.07 49.53 90) (unit 1)
     (in_bom yes) (on_board yes)
-    (property "Reference" "R?" (id 0) (at 175.26 46.99 90))
+    (property "Reference" "R11" (id 0) (at 175.26 46.99 90))
     (property "Value" "47K" (id 1) (at 179.07 46.99 90))
     (property "Footprint" "R_Resistor:R_0603" (id 2) (at 179.07 52.07 90)
@@
   (symbol (lib_id "R_Resistor:R_0603") (at 157.48 80.01 0) (unit 1)
     (in_bom yes) (on_board yes) (fields_autoplaced)
-    (property "Reference" "R?" (id 0) (at 159.131 78.2607 0)
+    (property "Reference" "R9" (id 0) (at 159.131 78.2607 0)
       (effects (font (size 1.27 1.27)) (justify left))
     )
@@
   (symbol (lib_id "R_Resistor:R_0603") (at 104.14 80.01 0) (unit 1)
     (in_bom yes) (on_board yes) (fields_autoplaced)
-    (property "Reference" "R?" (id 0) (at 105.791 78.2607 0)
+    (property "Reference" "R7" (id 0) (at 105.791 78.2607 0)
       (effects (font (size 1.27 1.27)) (justify left))
     )
@@
   (symbol (lib_id "power:GND") (at 157.48 91.44 0) (unit 1)
     (in_bom yes) (on_board yes) (fields_autoplaced)
-    (property "Reference" "#PWR?" (id 0) (at 157.48 97.79 0)
+    (property "Reference" "#PWR030" (id 0) (at 157.48 97.79 0)
       (effects (font (size 1.27 1.27)) hide)
     )
@@
   (symbol (lib_id "R_Resistor:R_0603") (at 96.52 80.01 0) (unit 1)
     (in_bom yes) (on_board yes) (fields_autoplaced)
-    (property "Reference" "R?" (id 0) (at 98.171 78.2607 0)
+    (property "Reference" "R6" (id 0) (at 98.171 78.2607 0)
       (effects (font (size 1.27 1.27)) (justify left))
     )
@@
   (symbol (lib_id "C_Capacitor:C_0603") (at 130.81 64.77 0) (unit 1)
     (in_bom yes) (on_board yes) (fields_autoplaced)
-    (property "Reference" "C?" (id 0) (at 133.1341 63.027 0)
+    (property "Reference" "C15" (id 0) (at 133.1341 63.027 0)
       (effects (font (size 1.27 1.27)) (justify left))
     )
@@
   (symbol (lib_id "R_Resistor:R_0603") (at 165.1 80.01 0) (unit 1)
     (in_bom yes) (on_board yes) (fields_autoplaced)
-    (property "Reference" "R?" (id 0) (at 166.751 78.2607 0)
+    (property "Reference" "R10" (id 0) (at 166.751 78.2607 0)
       (effects (font (size 1.27 1.27)) (justify left))
     )
@@
   (symbol (lib_id "R_Resistor:R_0603") (at 149.86 80.01 0) (unit 1)
     (in_bom yes) (on_board yes) (fields_autoplaced)
-    (property "Reference" "R?" (id 0) (at 151.511 78.2607 0)
+    (property "Reference" "R8" (id 0) (at 151.511 78.2607 0)
       (effects (font (size 1.27 1.27)) (justify left))
     )
@@
   (symbol (lib_id "C_Capacitor:C_0603") (at 118.11 54.61 0) (unit 1)
     (in_bom yes) (on_board yes) (fields_autoplaced)
-    (property "Reference" "C?" (id 0) (at 120.4341 52.867 0)
-      (effects (font (size 1.27 1.27)) (justify left))
-    )
+    (property "Reference" "C13" (id 0) (at 120.4341 52.867 0)
+      (effects (font (size 1.27 1.27)) (justify left))
+    )
